File: pcb/revA/zx-unikeyboard-ps2.kicad_pcb (KiCad board)
At the start: 2 copper layers, 79.2 x 17.8 mm, 13 parts, among them J1 MATRIX, J2 UART, J3 ISP, J4 PS/2, U1 ATmega32A-AU

Commit message: Small improvements to PCB rev.A
Parts:
- added REF**: KiCad-Logo2_8mm_SilkScreen, Symbol:KiCad-Logo2_8mm_SilkScreen, B.Cu at (103.9, 59.7)
- added REF**: WEEE-Logo_5.6x8mm_SilkScreen, Symbol:WEEE-Logo_5.6x8mm_SilkScreen, F.Cu at (138.2, 59.9)
- J4: footprint Connector_PinSocket_2.00mm:PinSocket_1x05_P2.00mm_Horizontal -> Connector_JST:JST_PH_S5B-PH-K_1x05_P2.00mm_Horizontal
- moved C2 1.48 mm to (142.5, 61.2), turned to 90 degrees
- moved J4 0.36 mm to (152.4, 66.3), turned to 90 degrees
Routing:
- net /PIN1: track 58.8 -> 57.3 mm
- net +5V: track 57.6 -> 58.2 mm, vias 2 -> 3
- net GND: vias 19 -> 26
Other:
- board text added: "CLK"
- board text added: "DAT"
- board text added: "rev.A"
