File: pcb/revA/zx-unikeyboard-ps2.sch (KiCad schematic (older format))
At the start: 13 parts, among them J1 MATRIX, J2 UART, J3 ISP, J4 PS/2, U1 ATmega32A-AU

Commit message: Small improvements to PCB rev.A
Parts:
- J4: footprint Connector_PinSocket_2.00mm:PinSocket_1x05_P2.00mm_Horizontal -> Connector_JST:JST_PH_S5B-PH-K_1x05_P2.00mm_Horizontal
Changed lines of the file:
@@
 F 0 "J4" H 8280 5042 50  0000 L CNN
 F 1 "PS/2" H 8280 4951 50  0000 L CNN
-F 2 "Connector_PinSocket_2.00mm:PinSocket_1x05_P2.00mm_Horizontal" H 8200 5000 50  0001 C CNN
+F 2 "Connector_JST:JST_PH_S5B-PH-K_1x05_P2.00mm_Horizontal" H 8200 5000 50  0001 C CNN
 F 3 "~" H 8200 5000 50  0001 C CNN
 	1    8200 5000
@@
 Text Label 7600 1550 0    50   ~ 0
 AVR_SS
-Wire Bus Line
-	7500 1300 7500 5600
-Wire Bus Line
-	5900 1300 5900 5150
 $Comp
 L Mechanical:MountingHole H1
@@
 	1    0    0    -1
 $EndComp
+Wire Bus Line
+	7500 1300 7500 5600
+Wire Bus Line
+	5900 1300 5900 5150
 $EndSCHEMATC
