File: pcb/revK/zx-unikeyboard-ps2.kicad_pcb (KiCad board)
At the start: 2 copper layers, 62 x 20.2 mm, 15 parts, among them J1 Matrix, J2 UART, J3 ISP, J4 Ext D, J5 Matrix, U1 ATmega32A-AU

Commit message: Updated PCB
Parts:
- moved REF** 2.03 mm to (124.2, 59.4)
- moved G*** 0.80 mm to (96.8, 60.2)
Routing:
- net /PIN26: track 37.4 -> 36.8 mm
- net /RESET: track 17.3 -> 17.8 mm
- net GND: track 6.71 -> 7.01 mm, vias 21 -> 18
Other:
- board text added: "CLK"
- board text added: "DAT"
- board text added: "PS/2"
